Commit message: Changed 'ec' to 'msl'.

File: msl_rotors_description/urdf/firefly_and_ball_base.xacro (robot description, xacro)
@@ -17,7 +17,7 @@
 -->
 <robot name="firefly" xmlns:xacro="http://ros.org/wiki/xacro">
-  <xacro:include filename="$(find ec_rotors_description)/urdf/component_snippets.xacro" />
+  <xacro:include filename="$(find msl_rotors_description)/urdf/component_snippets.xacro" />
   <!-- Instantiate firefly "mechanics" -->
-  <xacro:include filename="$(find ec_rotors_description)/urdf/firefly_and_ball.xacro" />
+  <xacro:include filename="$(find msl_rotors_description)/urdf/firefly_and_ball.xacro" />
   <!-- Instantiate a controller. -->
   <xacro:controller_plugin_macro namespace="${namespace}" imu_sub_topic="imu" />

File: msl_rotors_description/urdf/hummingbird_ball.xacro (robot description, xacro)
@@ -22,8 +22,8 @@
   <xacro:property name="rotor_velocity_slowdown_sim" value="10" />
   <xacro:property name="use_mesh_file" value="true" />
-  <xacro:property name="mesh_file" value="package://ec_rotors_description/meshes/hummingbird_ball_top.dae" />
-  <!-- <xacro:property name="mesh_file" value="package://ec_rotors_description/meshes/hummingbird_ball_only.dae" /> -->
-  <!-- <xacro:property name="mesh_file" value="package://ec_rotors_description/meshes/hummingbird_ball_center.dae" /> -->
-  <!-- <xacro:property name="mesh_file" value="package://ec_rotors_description/meshes/hummingbird_ball_bottom.dae" /> -->
+  <xacro:property name="mesh_file" value="package://msl_rotors_description/meshes/hummingbird_ball_top.dae" />
+  <!-- <xacro:property name="mesh_file" value="package://msl_rotors_description/meshes/hummingbird_ball_only.dae" /> -->
+  <!-- <xacro:property name="mesh_file" value="package://msl_rotors_description/meshes/hummingbird_ball_center.dae" /> -->
+  <!-- <xacro:property name="mesh_file" value="package://msl_rotors_description/meshes/hummingbird_ball_bottom.dae" /> -->
   <xacro:property name="mass" value="0.68" /> <!-- [kg] -->
   <xacro:property name="body_width" value="0.1" /> <!-- [m] -->
@@ -50,5 +50,5 @@
   </xacro:property>
   <!-- Included URDF Files -->
-  <xacro:include filename="$(find ec_rotors_description)/urdf/multirotor_base.xacro" />
+  <xacro:include filename="$(find msl_rotors_description)/urdf/multirotor_base.xacro" />
   <!-- Instantiate multirotor_base_macro once -->
   <xacro:multirotor_base_macro

File: msl_rotors_description/urdf/hummingbird_ball_base.xacro (robot description, xacro)
@@ -17,7 +17,7 @@
 -->
 <robot name="hummingbird" xmlns:xacro="http://ros.org/wiki/xacro">
-  <xacro:include filename="$(find ec_rotors_description)/urdf/component_snippets.xacro" />
+  <xacro:include filename="$(find msl_rotors_description)/urdf/component_snippets.xacro" />
   <!-- Instantiate hummingbird "mechanics" -->
-  <xacro:include filename="$(find ec_rotors_description)/urdf/hummingbird_ball.xacro" />
+  <xacro:include filename="$(find msl_rotors_description)/urdf/hummingbird_ball.xacro" />
   <!-- Instantiate a controller. -->
   <xacro:controller_plugin_macro namespace="${namespace}" imu_sub_topic="imu" />
